File: PCB/sourceFiles/rightside.kicad_sch (KiCad schematic)
At the start: 64 parts, among them SW27 SW_Push, SW28 SW_Push, SW29 SW_Push, SW30 SW_Push, SW31 SW_Push, SW32 SW_Push, SW33 SW_Push, SW34 SW_Push, SW35 SW_Push, SW36 SW_Push, SW37 SW_Push, SW38 SW_Push, SW39 SW_Push, SW40 SW_Push, SW41 SW_Push, SW42 SW_Push, SW43 SW_Push, SW44 SW_Push, SW45 SW_Push, SW46 SW_Push, SW47 SW_Push, SW48 SW_Push, SW49 SW_Push, SW50 SW_Push, SW51 SW_Push, SW52 SW_Push, U2 XIAO-nRF52840-SMD

Commit message: updated PCB from KiCad sourcs and gerbers
Connections:
- net R.col0: no longer D30.1 (K), D34.1 (K), D38.1 (K), D42.1 (K), D46.1 (K), D51.1 (K), SW31.1, SW32.1, SW33.1, SW34.1, SW35.1, SW36.1, SW37.1, SW38.1, SW39.1, SW40.1, SW41.1, SW42.1, SW43.1, SW44.1, SW45.1, SW46.1, SW52.1, U2.10 (P1.14_D9_MISO), U2.2 (P0.03_A1_D1), U2.3 (P0.28_A2_D2), U2.4 (P0.29_A3_D3), U2.5 (P0.04_A4_D4_SDA)
- net R.row0: now also U2.11 (P1.15_D10_MOSI); no longer U2.7 (P1.11_D6_TX)
- net R.row1: now also U2.10 (P1.14_D9_MISO); no longer U2.8 (P1.12_D7_RX)
- net R.row4: now also U2.7 (P1.11_D6_TX); no longer U2.11 (P1.15_D10_MOSI)
- new net R.col1: SW31.1, SW32.1, SW33.1, SW34.1, SW52.1, U2.2 (P0.03_A1_D1)
- new net R.col2: SW35.1, SW36.1, SW37.1, SW38.1, U2.3 (P0.28_A2_D2)
- new net R.col3: SW39.1, SW40.1, SW41.1, SW42.1, U2.4 (P0.29_A3_D3)
- new net R.col4: SW43.1, SW44.1, SW45.1, SW46.1, U2.5 (P0.04_A4_D4_SDA)
- new net R.row3: D30.1 (K), D34.1 (K), D38.1 (K), D42.1 (K), D46.1 (K), D51.1 (K), U2.8 (P1.12_D7_RX)
