File: PCB/sourceFiles/side.kicad_sch (KiCad schematic)
At the start: 64 parts, among them SW1 SW_Push, SW10 SW_Push, SW11 SW_Push, SW12 SW_Push, SW13 SW_Push, SW14 SW_Push, SW15 SW_Push, SW16 SW_Push, SW17 SW_Push, SW18 SW_Push, SW19 SW_Push, SW2 SW_Push, SW20 SW_Push, SW21 SW_Push, SW22 SW_Push, SW23 SW_Push, SW24 SW_Push, SW25 SW_Push, SW26 SW_Push, SW3 SW_Push, SW4 SW_Push, SW5 SW_Push, SW6 SW_Push, SW7 SW_Push, SW8 SW_Push, SW9 SW_Push, U1 XIAO-nRF52840-SMD

Commit message: updated PCB from KiCad sourcs and gerbers
Parts:
- added TP5, TP6: TestPoint, TestPoint:TestPoint_Pad_1.0x1.0mm, symbol Connector:TestPoint
Connections:
- net row0 is gone; now on net row1: D1.1 (K), D13.1 (K), D17.1 (K), D22.1 (K), D5.1 (K), D9.1 (K), U1.7 (P1.11_D6_TX)
- net col4: now also SW13.1, SW14.1, SW15.1, SW16.1, U1.4 (P0.29_A3_D3); no longer SW17.1, SW18.1, SW19.1, SW20.1, SW21.1, U1.5 (P0.04_A4_D4_SDA)
- net col5: now also SW17.1, SW18.1, SW19.1, SW20.1, SW21.1, U1.5 (P0.04_A4_D4_SDA); no longer SW22.1, SW23.1, SW24.1, SW25.1, SW26.1, U1.6 (P0.05_A5_D5_SCL)
- net row1: no longer D10.1 (K), D14.1 (K), D18.1 (K), D2.1 (K), D23.1 (K), D6.1 (K), U1.8 (P1.12_D7_RX)
- net row2: now also D10.1 (K), D14.1 (K), D18.1 (K), D2.1 (K), D23.1 (K), D6.1 (K), U1.8 (P1.12_D7_RX); no longer D11.1 (K), D15.1 (K), D19.1 (K), D24.1 (K), D3.1 (K), D7.1 (K), U1.9 (P1.13_D8_SCK)
- net row4: now also D12.1 (K), D16.1 (K), D20.1 (K), D25.1 (K), D4.1 (K), D8.1 (K), U1.10 (P1.14_D9_MISO); no longer D21.1 (K), D26.1 (K), U1.11 (P1.15_D10_MOSI)
- removed net col0: D12.1 (K), D16.1 (K), D20.1 (K), D25.1 (K), D4.1 (K), D8.1 (K), SW1.1, SW10.1, SW11.1, SW12.1, SW13.1, SW14.1, SW15.1, SW16.1, SW2.1, SW3.1, SW4.1, SW5.1, SW6.1, SW7.1, SW8.1, SW9.1, U1.1 (P0.02_A0_D0), U1.10 (P1.14_D9_MISO), U1.2 (P0.03_A1_D1), U1.3 (P0.28_A2_D2), U1.4 (P0.29_A3_D3)
- new net: TP5.1, TP6.1
- new net col1: SW1.1, SW2.1, SW3.1, SW4.1, U1.1 (P0.02_A0_D0)
- new net col2: SW5.1, SW6.1, SW7.1, SW8.1, U1.2 (P0.03_A1_D1)
- new net col3: SW10.1, SW11.1, SW12.1, SW9.1, U1.3 (P0.28_A2_D2)
- new net col6: SW22.1, SW23.1, SW24.1, SW25.1, SW26.1, U1.6 (P0.05_A5_D5_SCL)
- new net row3: D11.1 (K), D15.1 (K), D19.1 (K), D24.1 (K), D3.1 (K), D7.1 (K), U1.9 (P1.13_D8_SCK)
- new net row5: D21.1 (K), D26.1 (K), U1.11 (P1.15_D10_MOSI)
