File: PCB/sourceFiles/splitKey.kicad_pcb (KiCad board)
At the start: 2 copper layers, 290.8 x 123.8 mm, 125 parts, among them SW1 SW_Push, SW10 SW_Push, SW11 SW_Push, SW12 SW_Push, SW13 SW_Push, SW14 SW_Push, SW15 SW_Push, SW16 SW_Push, SW17 SW_Push, SW18 SW_Push, SW19 SW_Push, SW2 SW_Push, SW20 SW_Push, SW21 SW_Push, SW22 SW_Push, SW23 SW_Push, SW24 SW_Push, SW25 SW_Push, SW26 SW_Push, SW27 SW_Push, SW28 SW_Push, SW29 SW_Push, SW3 SW_Push, SW30 SW_Push, SW31 SW_Push, SW32 SW_Push, SW33 SW_Push, SW34 SW_Push, SW35 SW_Push, SW36 SW_Push, SW37 SW_Push, SW38 SW_Push, SW39 SW_Push, SW4 SW_Push, SW40 SW_Push, SW41 SW_Push, SW42 SW_Push, SW43 SW_Push, SW44 SW_Push, SW45 SW_Push, SW46 SW_Push, SW47 SW_Push, SW48 SW_Push, SW49 SW_Push, SW5 SW_Push, SW50 SW_Push, SW51 SW_Push, SW52 SW_Push, SW6 SW_Push, SW7 SW_Push, SW8 SW_Push, SW9 SW_Push, U1 XIAO-nRF52840-SMD, U2 XIAO-nRF52840-SMD

Commit message: updated PCB from KiCad sourcs and gerbers
Parts:
- added TP5: TestPoint, TestPoint:TestPoint_Pad_1.0x1.0mm, F.Cu at (165.9, 178.1)
- added TP6: TestPoint, TestPoint:TestPoint_Pad_1.0x1.0mm, F.Cu at (181.0, 178.0)
- turned D14 to 0 degrees
- turned D15 to 0 degrees
- turned D21 to 0 degrees
- turned D47 to 0 degrees
Connections:
- net col4 renamed /left/col5
- net col5 renamed /left/col6
- net row0 renamed /left/row1
- net row1 renamed /left/row2
- net row2 renamed /left/row3
- net row4 renamed /left/row5
- D12 pad 1: col0 -> /left/row4
- D16 pad 1: col0 -> /left/row4
- D20 pad 1: col0 -> /left/row4
- D25 pad 1: col0 -> /left/row4
- D30 pad 1: R.col0 -> R.row3
- D34 pad 1: R.col0 -> R.row3
- D38 pad 1: R.col0 -> R.row3
- D4 pad 1: col0 -> /left/row4
- D42 pad 1: R.col0 -> R.row3
- D46 pad 1: R.col0 -> R.row3
- D51 pad 1: R.col0 -> R.row3
- D8 pad 1: col0 -> /left/row4
- SW1 pad 1: col0 -> /left/col1
- SW10 pad 1: col0 -> /left/col3
- SW11 pad 1: col0 -> /left/col3
- SW12 pad 1: col0 -> /left/col3
- SW13 pad 1: col0 -> /left/col4
- SW14 pad 1: col0 -> /left/col4
- SW15 pad 1: col0 -> /left/col4
- SW16 pad 1: col0 -> /left/col4
- SW2 pad 1: col0 -> /left/col1
- SW3 pad 1: col0 -> /left/col1
- SW31 pad 1: R.col0 -> R.col1
- SW32 pad 1: R.col0 -> R.col1
- SW33 pad 1: R.col0 -> R.col1
- SW34 pad 1: R.col0 -> R.col1
- SW35 pad 1: R.col0 -> R.col2
- SW36 pad 1: R.col0 -> R.col2
- SW37 pad 1: R.col0 -> R.col2
- SW38 pad 1: R.col0 -> R.col2
- SW39 pad 1: R.col0 -> R.col3
- SW4 pad 1: col0 -> /left/col1
- SW40 pad 1: R.col0 -> R.col3
- SW41 pad 1: R.col0 -> R.col3
- SW42 pad 1: R.col0 -> R.col3
- SW43 pad 1: R.col0 -> R.col4
- SW44 pad 1: R.col0 -> R.col4
- SW45 pad 1: R.col0 -> R.col4
- SW46 pad 1: R.col0 -> R.col4
- SW5 pad 1: col0 -> /left/col2
- SW52 pad 1: R.col0 -> R.col1
- SW6 pad 1: col0 -> /left/col2
- SW7 pad 1: col0 -> /left/col2
- SW8 pad 1: col0 -> /left/col2
- SW9 pad 1: col0 -> /left/col3
- U1 pad 1: col0 -> /left/col1
- U1 pad 10: col0 -> /left/row4
- U1 pad 2: col0 -> /left/col2
- U1 pad 3: col0 -> /left/col3
- U1 pad 4: col0 -> /left/col4
- U2 pad 10: R.col0 -> R.row1
- U2 pad 11: R.row4 -> R.row0
- U2 pad 2: R.col0 -> R.col1
- U2 pad 3: R.col0 -> R.col2
- U2 pad 4: R.col0 -> R.col3
- U2 pad 5: R.col0 -> R.col4
- U2 pad 7: R.row0 -> R.row4
- U2 pad 8: R.row1 -> R.row3
Routing:
- net col0: track 438.6 -> 0.00 mm, vias 3 -> 0
- net R.col0: track 528.0 -> 122.4 mm
- net /left/row4: track 0.00 -> 191.5 mm, vias 0 -> 1
- net R.row3: track 0.00 -> 189.2 mm, vias 0 -> 1
- net R.col4: track 0.00 -> 186.1 mm
- net /left/col1: track 0.00 -> 169.1 mm
- net R.col3: track 0.00 -> 161.5 mm
- net /left/col2: track 0.00 -> 150.0 mm
- net R.col1: track 0.00 -> 144.0 mm
- net R.col2: track 0.00 -> 136.1 mm
- net /left/col3: track 0.00 -> 130.3 mm
- net /left/col4: track 0.00 -> 108.1 mm
- net R.GND: track 62.7 -> 29.2 mm
- net R.row2: track 157.7 -> 178.1 mm
- net R.row0: track 137.3 -> 119.6 mm
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- removed copper zone on B.Cu, net (none)
- removed copper zone on F.Cu, net (none)
Other:
- outline, holes or cut-outs redrawn
